File: espresif.kicad_sch (KiCad schematic)
At the start: 4 parts

Commit message: update: now the pcb has sheets and pcb layout
Parts:
- removed H1, H2, H3, H4: M3 screw, MountingHole:MountingHole_3.2mm_M3_DIN965_Pad, symbol Mechanical:MountingHole_Pad
- added B1, B2: ~, JuanDavid_Library:SW-SMD_L3.9-W2.9-LS4.8, symbol JuanDavid_Library:SlimButton
- added C5, C6: 100nF, Capacitor_SMD:C_0603_1608Metric, symbol Device:C
- added J1: UART, Connector_PinSocket_2.54mm:PinSocket_1x03_P2.54mm_Vertical, symbol Connector:Conn_01x03_Pin
- added R10, R9: 3.3K, Resistor_SMD:R_0603_1608Metric, symbol Device:R_US
- added U1: ~, JuanDavid_Library:WIFI-SMD_ESP32-WROOM-32E, symbol JuanDavid_Library:ESP32-WROOM-32E-N8
Connections:
- net GND: now also B1.1, B2.1, C5.2, C6.2, J1.3 (Pin_3), U1.1 (GND), U1.15 (GND), U1.38 (GND), U1.39 (GND)
- new net +3.3V: R10.1, R9.1, U1.2 (3V3)
- new net Boot: B2.2, C6.1, R10.2, U1.25 (IO0)
- new net CLK: U1.13 (IO14)
- new net CS: U1.23 (IO15)
- new net CS_{T}: U1.30 (IO18)
- new net D0: U1.26 (IO4)
- new net D/C: U1.24 (IO2)
- new net EN: B1.2, C5.1, R9.2, U1.3 (EN)
- new net LED: U1.33 (IO21)
- new net MISO: U1.14 (IO12)
- new net MOSI: U1.16 (IO13)
- new net RST: U1.29 (IO5)
- new net Rx: J1.2 (Pin_2), U1.35 (TXD0)
- new net SCK: U1.36 (IO22)
- new net T_CLK: U1.10 (IO25)
- new net T_CS: U1.9 (IO33)
- new net T_DIN: U1.8 (IO32)
- new net T_DO: U1.5 (SENSOR_VN)
- new net T_IRQ: U1.4 (SENSOR_VP)
- new net TriggerGate: U1.27 (IO16)
- new net Tx: J1.1 (Pin_1), U1.34 (RXD0)
- new net zero_cross: U1.6 (IO34)
Other:
- removed sheet Power
- removed sheet esp32
- removed sheet modules
- note added: "Boot and reset buttons"
- note added: "UART pins"
- note removed: "M3 screw"
- note removed: "Modules"
- note removed: "POWER"
- title: Solder Oven -> (none)

Commit message: update: pcb with component in place
Connections:
- no-connect marks 0 -> 7
Changed lines of the file:
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@@
 		(color 0 0 0 0)
+	)
+	(no_connect
+		(at 65.913 63.246)
+	)
+	(no_connect
+		(at 65.913 40.386)
+	)
+	(no_connect
+		(at 35.433 53.086)
+	)
+	(no_connect
+		(at 65.913 55.626)
+	)
+	(no_connect
+		(at 35.433 63.246)
+	)
+	(no_connect
+		(at 65.913 53.086)
+	)
+	(no_connect
+		(at 35.433 65.786)
 	)
 	(wire
