File: modules.kicad_sch (KiCad schematic)
At the start: 15 parts, among them U4 H11AA1, U5 MOC3052M

Commit message: update: gerbers generator
Parts:
- added C8: 100n, Capacitor_THT:C_Disc_D5.0mm_W2.5mm_P2.50mm, symbol Device:C_Polarized_Small_US
- added R12: 150, Resistor_THT:R_Axial_DIN0204_L3.6mm_D1.6mm_P5.08mm_Horizontal, symbol Device:R_US
Connections:
- net shot: now also C8.1, R12.1
- net at D1.1 (A1), R1.1: now also C8.2, R12.2
